File: mikrainix/SPLink.kicad_sch (KiCad schematic)
At the start: 72 parts, among them J1 2345986-1, J2 Conn_01x04_Socket, Q1 STL6P3LLH6, Q2 STL6P3LLH6, SW1 SW_Push, U1 STUSB4500QTR, U2 ST1S40IPUR, U3 STM32L052C8U6, U4 L7983PUR, U5 ECMF02-2AMX6, Y1 FY1600069Q (16 MHZ)

Commit message: update SPLink schematic
Parts:
- removed C10: 27p, symbol Device:C
- removed C11: 22µ, symbol Device:C
- removed C15: 100n, symbol Device:C
- removed D1, D3, D5: 824045812, symbol Device:D_Zener
- removed D4: (x2) 824045812, symbol Device:D_Zener
- removed D6: LED, symbol Device:LED
- removed F1: MF-LSMF300/16X, symbol Device:Polyfuse
- removed R15: 3.3k, symbol Device:R
- removed R16: 1k, symbol Device:R
- removed R7: 68k, symbol Device:R
- removed R9: 13k, symbol Device:R
- removed U2: ST1S40IPUR, mikrainix-ST1S40IPUR:QFPN_40IPUR_STM, symbol mikrainix-ST1S40IPUR:ST1S40IPUR
- added C29, C30, C31: 1µ, symbol Device:C
- added C32: 100n, symbol Device:C
- added C33: 68µ, symbol Device:C
- added C34: 9.1p, symbol Device:C
- added CR1, CR2: ESDA25P35-1U1M, mikrainix-ESDA25P35-1U1M:QFN1610_STM, symbol mikrainix-ESDA25P35:ESDA25P35-1U1M
- added CR3: ESDA25W, mikrainix-ESDA25W:SOT323-3L_STM, symbol mikrainix-ESDA25W:ESDA25W
- added D10, D8, D9: LED, symbol Device:LED
- added Q3, Q4: 2N7002, Package_TO_SOT_SMD:SOT-23, symbol Transistor_FET:2N7002
- added R23: 100, symbol Device:R
- added R24, R25, R28: 1k, symbol Device:R
- added R26, R27: 10k, symbol Device:R
- added U2: L6983N50QTR, WFQFN16_3X3X0P5_STM, symbol mikrainix-L6983N50QTR:L6983N50QTR
- C14: value 4.7µ -> 1µ
- C21: value 10µ -> 4.7µ
- C22: value 22p -> 100n
- L1: value 4.7µ -> 12µ
- L2: value 82µ -> 33µ
Connections:
- net 3V3: now also C22.2, R18.2, C34.2, R24.2, R27.2, R28.2; no longer C22.1, R18.1
- net 5V: now also C33.1, R25.2, R26.2, U2.7 (FB/VOUT)
- net CC1: now also CR3.1
- net CC2: now also CR3.2
- net GND: now also C22.1, U4.4 (FSW), C29.2, C30.2, C31.2, C33.2, CR1.2, CR2.2, CR3.3, Q3.2 (S), Q4.2 (S), U2.10 (AGND), U2.13 (PGND), U2.16 (PGND), U2.17 (EPAD), U2.3 (AGND), U2.6 (VBIAS), U2.8 (FSW)
- net LED1: now also Q3.1 (G), R26.1, U2.5 (PGOOD); no longer D7.1 (K), U3.38 (PA15)
- net VBUS: now also CR1.1
- net VPSNK: now also C8.1, C9.1, C29.1, CR2.1, R23.1, U2.1 (VIN), U2.12 (VIN), U2.4 (EN/CLKIN)
- net LED3: now reaches U3.10 (PA0)
- net LED3: now also D7.1 (K)
- net LED4: now reaches U3.11 (PA1)
- net LED4: now also D8.1 (K)
- net at L1.1: now also C32.1, U2.14 (SW), U2.15 (SW)
- net at D7.2 (A): now also R18.1; no longer R18.2
- net at R14.2, R17.1, U4.1 (VOUT/FB): now also C34.1; no longer C22.2
- net LED0 renamed LED2
- net LED2: now also Q4.1 (G), R27.1
- new net: D8.2 (A), R24.1
- new net: D9.2 (A), R25.1
- new net: D9.1 (K), Q3.3 (D)
- new net: C30.1, R23.2, U2.2 (VINLDO)
- new net: D10.2 (A), R28.1
- new net: D10.1 (K), Q4.3 (D)
- new net: C32.2, U2.11 (BOOT)
- new net: C31.1, U2.9 (VCC)
- no-connect marks 35 -> 34
Other:
- moved on the sheet: C1, C12, C13, C14, C16, C17, C18, C19, C2, C20, C21, C23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

Commit message: add USB WiFi and update MPU RV1106G3 schematics
Parts:
- removed C17, C18: 100n, symbol Device:C
- removed U5: ECMF02-2AMX6, mikrainix-ECMF02-2AMX6:QFN-6L_STM, symbol mikrainix-ECMF02-2AMX6:ECMF02-2AMX6
- added C24, C25, C26, C27: 100n, symbol Device:C
- added C31: 10n, symbol Device:C
- added R13, R23, R24: 10k, symbol Device:R
- added SW2: BUSB, symbol Switch:SW_Push
- added U5: MAX4899EETE+T, mikrainix-MAX4899EETE-T:21-0136_T1633+4_MXM, symbol mikrainix-MAX4899EETE-T:MAX4899EETE+T
- added U6: ECMF02-2AMX6, mikrainix-ECMF02-2AMX6:QFN-6L_STM, symbol mikrainix-ECMF02-2AMX6:ECMF02-2AMX6
- C30: renamed from C25; value 10n -> 10µ; now not fitted
- C32: renamed from C26; value 10µ -> 100n; now fitted
- SW1: value SW_Push -> BRESET
- Y1: value FY1600069Q (16 MHZ) -> 16 MHz
- renumbered C8 to C10, C9 to C11, C29 to C12, C12 to C13, C30 to C14, C31 to C15, C13 to C16, C14 to C17, C21 to C18, C23 to C20, C34 to C21, C16 to C23, C20 to C28, C24 to C29, C27 to C33, C28 to C34, C32 to C7, C33 to C8, C7 to C9, D2 to D1, D9 to D2, D10 to D3, D7 to D4, D8 to D5, R11 to R10, R12 to R11, R13 to R12, R17 to R15, R26 to R16, R25 to R17, R27 to R18, R28 to R19, R18 to R20, R24 to R21, R19 to R22, R20 to R25, R21 to R26, R22 to R27, R8 to R7, R23 to R8, R10 to R9
Connections:
- net 3V3: now also C24.1, C25.1, C26.1, C27.1, R13.1, U5.4 (V+); no longer C19.1
- net DN1: now also U6.2 (D-)
- net DP1: now also U6.1 (D+)
- net GND: now also C24.2, C25.2, C26.2, C27.2, C31.2, R23.2, R24.2, SW2.1, U5.1 (GND), U5.15 (nEN), U5.16 (nQP), U5.17 (EPAD), U6.3 (GND)
- net VDDA: now also C31.1
- net BUSB: now reaches U3.15 (PA5)
- net BUSB: now also C19.1, R13.2, SW2.2
- net USB_C0: now reaches U3.16 (PA6)
- net USB_C0: now also R23.1, U5.6 (C0)
- net USB_C1: now reaches U3.17 (PA7)
- net USB_C1: now also R24.1, U5.5 (C1)
- net PS_MODE: now reaches U3.21 (PB10)
- net PS_EN1: now reaches U3.22 (PB11)
- net PS_EN2: now reaches U3.25 (PB12)
- net PS_EN3: now reaches U3.26 (PB13)
- net PS_LEN1: now reaches U3.27 (PB14)
- net PS_LEN2: now reaches U3.28 (PB15)
- net VBUS_DET: now reaches U3.29 (PA8)
- net COM.RX1 renamed RX1
- net COM.RX2 renamed RX2
- net COM.TX1 renamed TX1
- net COM.TX2 renamed TX2
- net D+ renamed MCU_D+
- net MCU_D+: now also U5.13 (USB0+)
- net D- renamed MCU_D-
- net MCU_D-: now also U5.14 (USB0-)
- net WKUP: no longer names the net of U3.2 (PC13)
- new net: U5.2 (COMA+), U6.6 (D+)
- new net: U5.3 (COMA-), U6.5 (D-)
- new net ESP_D+: U5.10 (USB2+)
- new net ESP_D-: U5.9 (USB2-)
- new net MPU_D+: U5.11 (USB1+)
- new net MPU_D-: U5.12 (USB1-)
- no-connect marks 34 -> 25
Other:
- note added: "COM. SERIAL UART"
- note added: "COM. USB"
- note added: "CTRL. POWER SUPPLY"
- note removed: "COM. SERIAL UART1"
- note removed: "COM. SERIAL UART2"
- note removed: "SYSTEM RESET"
- note removed: "SYSTEM WAKEUP"
- note removed: "USB DEVICE"
- moved on the sheet: C13, C23, C28, C29, C33, C34, FB1, J2, R10, R11, R12, R20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
