File: mikrainix/SPLink.kicad_sch (KiCad schematic)
At the start: 87 parts, among them J1 2345986-1, J2 Conn_01x04_Socket, Q1 STL6P3LLH6, Q2 STL6P3LLH6, Q3 2N7002, Q4 2N7002, SW1 BRESET, SW2 BUSB, U1 STUSB4500QTR, U2 L6983N50QTR, U3 STM32L052C8U6, U4 L7983PUR, U5 MAX4899EETE+T, U6 ECMF02-2AMX6, Y1 16 MHz

Commit message: add MIS5001 camera and Ethernet, replace ESP32-C6-MINI > ESP32-MINI-1
Parts:
- D1: value 1PS10SB82 -> BAT54JFILM
Changed lines of the file:
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@@
 			)
 		)
-		(property "Value" "1PS10SB82"
+		(property "Value" "BAT54JFILM"
 			(at 251.46 38.4174 90)
 			(show_name no)
@@
 			)
 		)
-		(property "Datasheet" ""
+		(property "Datasheet" "https://www.st.com/resource/en/datasheet/bat54.pdf"
 			(at 254 36.83 0)
 			(hide yes)

Commit message: add microSD and resolve ERC issues
Other:
- title: Smart Power Link v1.0 -> Smart Power Link
Changed lines of the file:
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@@
 	(paper "A3")
 	(title_block
-		(title "Smart Power Link v1.0")
-		(date "2026-10-08")
+		(title "Smart Power Link")
+		(date "2026-10-21")
+		(rev "v0.1")
 		(comment 1 "Project repository: github.com/ndkimdavy/Mikrainix")
 		(comment 2 "Designed by: Kim Davy NDAYONGEJE")
@@
 	)
 	(junction
-		(at 304.8 88.9)
-		(diameter 0)
-		(color 0 0 0 0)
-	)
-	(junction
 		(at 22.86 39.37)
 		(diameter 0)
@@
 		(in_pos_files yes)
 		(dnp no)
-		(property "Reference" "#FLG09"
+		(property "Reference" "#FLG08"
 			(at 194.31 239.395 0)
 			(hide yes)
@@
 			(project "mikrainix"
 				(path "/19082ed6-8f17-4d62-ab42-418ea03b55ea/22cc9e10-2568-472f-808f-2c6ffeb9eeb0"
-					(reference "#FLG09")
+					(reference "#FLG08")
 					(unit 1)
 				)
@@
 		(in_pos_files yes)
 		(dnp no)
-		(property "Reference" "#FLG05"
+		(property "Reference" "#FLG04"
 			(at 143.51 239.395 0)
 			(hide yes)
@@
 			(project "mikrainix"
 				(path "/19082ed6-8f17-4d62-ab42-418ea03b55ea/22cc9e10-2568-472f-808f-2c6ffeb9eeb0"
-					(reference "#FLG05")
+					(reference "#FLG04")
 					(unit 1)
 				)
@@
 		(in_pos_files yes)
 		(dnp no)
-		(property "Reference" "#FLG010"
+		(property "Reference" "#FLG09"
 			(at 207.01 239.395 0)
 			(hide yes)
@@
 			(project "mikrainix"
 				(path "/19082ed6-8f17-4d62-ab42-418ea03b55ea/22cc9e10-2568-472f-808f-2c6ffeb9eeb0"
-					(reference "#FLG010")
+					(reference "#FLG09")
 					(unit 1)
 				)
@@
 		(in_pos_files yes)
 		(dnp no)
-		(property "Reference" "#FLG04"
+		(property "Reference" "#FLG03"
 			(at 130.81 239.395 0)
 			(hide yes)
@@
 			(project "mikrainix"
 				(path "/19082ed6-8f17-4d62-ab42-418ea03b55ea/22cc9e10-2568-472f-808f-2c6ffeb9eeb0"
-					(reference "#FLG04")
+					(reference "#FLG03")
 					(unit 1)
 				)
@@
 		(in_pos_files yes)
 		(dnp no)
-		(property "Reference" "#FLG02"
+		(property "Reference" "#FLG01"
 			(at 304.8 97.155 0)
 			(hide yes)
@@
 			(project "mikrainix"
 				(path "/19082ed6-8f17-4d62-ab42-418ea03b55ea/22cc9e10-2568-472f-808f-2c6ffeb9eeb0"
-					(reference "#FLG02")
+					(reference "#FLG01")
 					(unit 1)
 				)
@@
 		(in_pos_files yes)
 		(dnp no)
-		(property "Reference" "#FLG08"
+		(property "Reference" "#FLG07"
 			(at 181.61 239.395 0)
 			(hide yes)
@@
 			(project "mikrainix"
 				(path "/19082ed6-8f17-4d62-ab42-418ea03b55ea/22cc9e10-2568-472f-808f-2c6ffeb9eeb0"
-					(reference "#FLG08")
+					(reference "#FLG07")
 					(unit 1)
 				)
@@
 		(in_pos_files yes)
 		(dnp no)
-		(property "Reference" "#FLG07"
+		(property "Reference" "#FLG06"
 			(at 168.91 239.395 0)
 			(hide yes)
@@
 			(project "mikrainix"
 				(path "/19082ed6-8f17-4d62-ab42-418ea03b55ea/22cc9e10-2568-472f-808f-2c6ffeb9eeb0"
-					(reference "#FLG07")
+					(reference "#FLG06")
 					(unit 1)
 				)
@@
 	)
 	(symbol
-		(lib_id "power:PWR_FLAG")
-		(at 304.8 88.9 0)
-		(unit 1)
-		(body_style 1)
-		(exclude_from_sim no)
-		(in_bom yes)
-		(on_board yes)
-		(in_pos_files yes)
-		(dnp no)
-		(property "Reference" "#FLG01"
-			(at 304.8 86.995 0)
-			(hide yes)
-			(show_name no)
-			(do_not_autoplace no)
-			(effects
-				(font
-					(size 1.27 1.27)
-				)
-			)
-		)
-		(property "Value" "PWRF"
-			(at 304.8 83.82 0)
-			(show_name no)
-			(do_not_autoplace no)
-			(effects
-				(font
-					(size 1.27 1.27)
-				)
-			)
-		)
-		(property "Footprint" ""
-			(at 304.8 88.9 0)
-			(hide yes)
-			(show_name no)
-			(do_not_autoplace no)
-			(effects
-				(font
-					(size 1.27 1.27)
-				)
-			)
-		)
-		(property "Datasheet" ""
-			(at 304.8 88.9 0)
-			(hide yes)
-			(show_name no)
-			(do_not_autoplace no)
-			(effects
-				(font
-					(size 1.27 1.27)
-				)
-			)
-		)
-		(property "Description" "Special symbol for telling ERC where power comes from"
-			(at 304.8 88.9 0)
-			(hide yes)
-			(show_name no)
-			(do_not_autoplace no)
-			(effects
-				(font
-					(size 1.27 1.27)
-				)
-			)
-		)
-		(pin "1"
-		)
-		(instances
-			(project "mikrainix"
-				(path "/19082ed6-8f17-4d62-ab42-418ea03b55ea/22cc9e10-2568-472f-808f-2c6ffeb9eeb0"
-					(reference "#FLG01")
-					(unit 1)
-				)
-			)
-		)
-	)
-	(symbol
 		(lib_id "Device:C")
 		(at 254 93.98 0)
@@
 		(in_pos_files yes)
 		(dnp no)
-		(property "Reference" "#FLG06"
+		(property "Reference" "#FLG05"
 			(at 156.21 239.395 0)
 			(hide yes)
@@
 			(project "mikrainix"
 				(path "/19082ed6-8f17-4d62-ab42-418ea03b55ea/22cc9e10-2568-472f-808f-2c6ffeb9eeb0"
-					(reference "#FLG06")
+					(reference "#FLG05")
 					(unit 1)
 				)
@@
 		(in_pos_files yes)
 		(dnp no)
-		(property "Reference" "#FLG03"
+		(property "Reference" "#FLG02"
 			(at 118.11 239.395 0)
 			(hide yes)
@@
 			(project "mikrainix"
 				(path "/19082ed6-8f17-4d62-ab42-418ea03b55ea/22cc9e10-2568-472f-808f-2c6ffeb9eeb0"
-					(reference "#FLG03")
+					(reference "#FLG02")
 					(unit 1)
 				)

Commit message: add ESD protection
Parts:
- removed CR1, CR2: ESDA25P35-1U1M, mikrainix-ESDA25P35-1U1M:QFN1610_STM, symbol mikrainix-ESDA25P35:ESDA25P35-1U1M
- removed CR3: ESDA25W, mikrainix-ESDA25W:SOT323-3L_STM, symbol mikrainix-ESDA25W:ESDA25W
- removed U1: STUSB4500QTR, mikrainix-STUSB4500QTR:QFN24EP_4X4_STM, symbol mikrainix-STUSB4500QTR:STUSB4500QTR
- removed U2: L6983N50QTR, WFQFN16_3X3X0P5_STM, symbol mikrainix-L6983N50QTR:L6983N50QTR
- removed U3: STM32L052C8U6, mikrainix-STM32L052C8U6:UFQFPN-48_STM, symbol mikrainix-STM32L052C8U6:STM32L052C8U6
- removed U6: ECMF02-2AMX6, mikrainix-ECMF02-2AMX6:QFN-6L_STM, symbol mikrainix-ECMF02-2AMX6:ECMF02-2AMX6
- added D1, D8: ESDA25P35-1U1M, mikrainix-ESDA25P35-1U1M:QFN1610_STM, symbol mikrainix-ESD_SYM:ESDx1
- added D2: ESDA25W, mikrainix-ESDA25W:SOT323-3L_STM, symbol mikrainix-ESD_SYM:ESDx2
- added D9: HSP051-2W3Y, mikrainix-HSP051-2W3Y:SOT323-3L_1P35X2P2X0P65_STM, symbol mikrainix-ESD_SYM:ESDx2
- added U1: STM32L052C8U6, mikrainix-STM32L052C8U6:UFQFPN-48_STM, symbol mikrainix-STM32L052C8U6:STM32L052C8U6
- added U2: STUSB4500QTR, mikrainix-STUSB4500QTR:QFN24EP_4X4_STM, symbol mikrainix-STUSB4500QTR:STUSB4500QTR
- added U3: ECMF02-2AMX6, mikrainix-ECMF02-2AMX6:QFN-6L_STM, symbol mikrainix-ECMF02-2AMX6:ECMF02-2AMX6
- added U6: L6983N50QTR, mikrainix-L6983N50QTR:WFQFN16_3X3X0P5_STM, symbol mikrainix-L6983N50QTR:L6983N50QTR
- C1: renamed from C23; value 4.7µ -> 100n
- C13: renamed from C28; value 100n -> 4.7µ
- C6: renamed from C30; value 10µ -> 10n; now fitted
- C9: renamed from C31; value 10n -> 10µ; now not fitted
- renumbered C3 to C10, C13 to C11, C19 to C12, C32 to C14, C34 to C15, C1 to C16, C2 to C17, C4 to C18, C9 to C19, C24 to C2, C6 to C20, C10 to C21, C16 to C22, C11 to C23, C17 to C24, C20 to C25, C12 to C26, C14 to C27, C15 to C28, C5 to C29, C25 to C3, C18 to C30, C21 to C31, C22 to C32, C7 to C33, C8 to C34, C29 to C4, C26 to C5, C33 to C7, C27 to C8, D2 to D3, D3 to D4, D4 to D5, D5 to D6, D1 to D7, L2 to L1, L1 to L2, Q3 to Q1, Q4 to Q2, Q1 to Q3, Q2 to Q4, R22 to R1, R18 to R10, R19 to R11, R20 to R12, R21 to R13, R1 to R14, R4 to R15, R5 to R16, R2 to R17, R6 to R18, R23 to R19, R25 to R2, R8 to R20, R24 to R21, R3 to R22, R14 to R23, R15 to R24, R9 to R25, R11 to R26, R10 to R27, R26 to R3, R7 to R4, R12 to R5, R13 to R6, R27 to R7, R16 to R8, R17 to R9
Connections:
- net 3V3: now also U1.1 (VDD), U1.24 (VDD), U1.36 (VDD_USB), U1.48 (VDD)
- net 5V: now also U6.7 (FB/VOUT)
- net ALERT: now also U1.41 (PB5), U2.19 (ALERT)
- net A_B_SIDE: now also U1.18 (PB0), U2.17 (A_B_SIDE)
- net BOOT0: now also U1.44 (BOOT0)
- net BUSB: now also U1.15 (PA5)
- net CC1: now also D2.1, U2.1 (CC1DB), U2.2 (CC1)
- net CC2: now also D2.2, U2.4 (CC2), U2.5 (CC2DB)
- net DISCH: now also U2.9 (DISCH)
- net DN1: now also U3.2 (D-)
- net DP1: now also U3.1 (D+)
- net GND: now also D1.2, D2.3, D8.2, D9.3, U1.23 (VSS), U1.35 (VSS), U1.47 (VSS), U1.49 (EPAD), U1.8 (VSSA), U2.10 (GND), U2.12 (ADDR0), U2.13 (ADDR1), U2.22 (VSYS), U2.25 (EPAD), U2.6 (RESET), U3.3 (GND), U6.10 (AGND), U6.13 (PGND), U6.16 (PGND), U6.17 (EPAD), U6.3 (AGND), U6.6 (VBIAS), U6.8 (FSW)
- net LED1: now also U6.5 (PGOOD)
- net LED3: now also U1.10 (PA0)
- net LED4: now also U1.11 (PA1)
- net MCU_D+: now also U1.33 (PA12)
- net MCU_D-: now also U1.32 (PA11)
- net NRST: now also U1.7 (NRST)
- net OSC_IN: now also U1.5 (PH0-OSC_IN)
- net OSC_OUT: now also U1.6 (PH1-OSC_OUT)
- net PS_EN1: now also U1.22 (PB11)
- net PS_EN2: now also U1.25 (PB12)
- net PS_EN3: now also U1.26 (PB13)
- net PS_LEN1: now also U1.27 (PB14)
- net PS_LEN2: now also U1.28 (PB15)
- net PS_MODE: now also U1.21 (PB10)
- net RX1: now also U1.31 (PA10)
- net RX2: now also U1.13 (PA3)
- net SCL: now also U1.42 (PB6), U2.7 (SCL)
- net SDA: now also U1.43 (PB7), U2.8 (SDA)
- net SWCLK: now also D9.2, U1.37 (PA14)
- net SWDIO: now also U1.34 (PA13)
- net TX1: now also U1.30 (PA9)
- net TX2: now also U1.12 (PA2)
- net USB_C0: now also U1.16 (PA6)
- net USB_C1: now also U1.17 (PA7)
- net VBUS: now also D1.1
- net VBUS_DET: now also U1.29 (PA8)
- net VBUS_EN_SNK: now also U2.16 (VBUS_EN_SNK)
- net VBUS_VS_DISCH: now also U2.18 (VBUS_VS_DISCH)
- net VDDA: now also U1.9 (VDDA)
- net VDD/VBUS: now also U2.24 (VDD)
- net VPSNK: now also D8.1, U6.1 (VIN), U6.12 (VIN), U6.4 (EN/CLKIN)
- net at J2.2 (Pin_2), R27.2: now also D9.1
- net at U5.2 (COMA+): now also U3.6 (D+)
- net at U5.3 (COMA-): now also U3.5 (D-)
- net at C33.1, L2.1: now also U6.14 (SW), U6.15 (SW)
- net at C17.1: now also U2.21 (VREG_1V2)
- net at C18.1: now also U2.23 (VREG_2V7)
- net at C27.1, R20.2: now also U6.2 (VINLDO)
- net at C33.2: now also U6.11 (BOOT)
- net at C28.1: now also U6.9 (VCC)
Other:
- note removed: "LEDx"
- note removed: "SERIAL WIRE DEBUG"
- moved on the sheet: C10, C16, C17, C18, C19, C20, C21, C22, C23, C24, C25, C26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
