File: mikrainix/MPU-USB-Wifi-Ethernet.kicad_sch (KiCad schematic)
At the start: 55 parts, among them Q6 2N7002, Q7 2N7002, Q8 2N7002, SW5 BEN, SW6 BFLASH, U10 ESP32-MINI-1, U11 CP2102N-A02-GQFN24, U7 RV1106G3, U9 TPS62821DLCR

Commit message: add ESD protection
Parts:
- removed C103, C104: 4.7µ, symbol Device:C
- removed U7: RV1106G3, mikrainix-RV1106G3:QFN35P1230X1230X90-129N, symbol mikrainix-RV1106G3:RV1106G3
- added C106, C107: 4.7µ, symbol Device:C
- added U8: RV1106G3, mikrainix-RV1106G3:QFN35P1230X1230X90-129N, symbol mikrainix-RV1106G3:RV1106G3
- renumbered C106 to C100, C102 to C101, C98 to C102, C96 to C103, C97 to C104, C107 to C96, C99 to C97, C100 to C98, C101 to C99, D9 to D11, D7 to D12, D8 to D13, Q7 to Q6, Q8 to Q7, Q6 to Q8, R69 to R54, R70 to R55, R76 to R56, R79 to R57, R71 to R58, R77 to R59, R78 to R60, R72 to R61, R73 to R62, R74 to R63, R81 to R64, R75 to R65, R80 to R66, R58 to R67, R62 to R68, R66 to R69, R67 to R70, R68 to R71, R63 to R72, R54 to R73, R55 to R74, R64 to R75, R65 to R76, R56 to R77, R59 to R78, R61 to R79, R57 to R80, R60 to R81, SW6 to SW5, SW5 to SW6
Connections:
- net 1SDIO_CLK: now also U8.93 (VO_LCDC_D5/VI_CIF_D4_M1/PWM5_M2/I2C4_SCL_M1/SDMMC1_CLK_M1/SPI0_MOSI_M0/GPIO1_C2_d)
- net 2MPU_D+: now also U8.27 (USB_DP)
- net 2MPU_D-: now also U8.26 (USB_DM)
- net 3V3/1A: now also C106.2, C107.2
- net GND: now also C106.1, C107.1
- net SDIO_CMD: now also U8.92 (VO_LCDC_D4/VI_CIF_D5_M1/PWM6_M2/I2C4_SDA_M1/SDMMC1_CMD_M1/SPI0_MISO_M0/GPIO1_C3_d)
- net SDIO_D0: now also U8.94 (VO_LCDC_D6/VI_CIF_D3_M1/PWM4_M2/SPI0_CLK_M0/SDMMC1_D0_M1/GPIO1_C1_d)
- net SDIO_D1: now also U8.95 (VO_LCDC_D7/VI_CIF_D2_M1/PWM2_M2/SPI0_CS0_M0/SDMMC1_D1_M1/GPIO1_C0_d)
- net SDIO_D2: now also U8.90 (VO_LCDC_D2/VI_CIF_D7_M1/PWM9_M1/UART4_TX_M1/SDMMC1_D2_M1/GPIO1_C5_d)
- net SDIO_D3: now also U8.91 (VO_LCDC_D3/VI_CIF_D6_M1/PWM8_M1/UART4_RX_M1/SDMMC1_D3_M1/GPIO1_C4_d)
- net at R77.2, R78.1: now also U8.25 (USB_VBUSDET)
Other:
- moved on the sheet: C100, C101, C102, C103, C104, C96, C97, C98, C99, D11, D12, D13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
